File: electronics/decant/decant.kicad_sch (KiCad schematic)
At the start: 56 parts, among them J1 USB_B, J2 Conn_01x03_Pin, J3 Conn_ARM_JTAG_SWD_10, J4 1985218, J5 Conn_01x03_Pin, SW1 PTS810_SJM_250_SMTR_LFS, U1 USBLC6-2SC6, U2 STM32F412RGTx, U3 TPS63001, U4 MCP2562-E-SN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

Commit message: working on filtered table and bit inspector
Other:
- note added: "LQH3NPN2R2MJRL"
Changed lines of the file:
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@@
     (stroke (width 0) (type default))
+  )
+  (text "LQH3NPN2R2MJRL" (at 92.075 192.405 90)
+    (effects (font (size 1.27 1.27)) (justify left bottom))
   )
   (text "1/4W" (at 83.185 163.83 0)
